Commit message: chore(repo): SerialArm-Core 更新至 v0.5.2，支持外部 profile_file/resource_paths

File: src/tomato_picker/description/urdf/tomato_picker.urdf (robot description, URDF)
Before this commit: robot Tomato-Picker, 10 links, 9 joints
Links:
- added link tool0
Joints:
- added joint tool0_joint: type fixed, parent Link6, child tool0, origin xyz=0 0 0 rpy=0 0 0

Commit message: feat(tomato-picker): update URDF and config for new model

File: src/tomato_picker/description/urdf/tomato_picker.urdf (robot description, URDF)
Before this commit: robot Tomato-Picker, 11 links, 10 joints
Links:
- link Link1: mass 0.089811 -> 0.0898108036954061
- link Link2: mass 0.9887 -> 1.07002287894776
- link Link3: mass 0.55814 -> 0.610419134840687
- link Link4: mass 0.34575 -> 0.345655632636913
- link Link5: mass 0.374 -> 0.373823984061805
- link Link6: mass 0.786 -> 0.785649631359557
- link Link7: mass 0.006 -> 0.00643315957914466; geometry collision mesh filename=package://tomato_picker_description/meshes/solidworks/Link7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; visual mesh filename=package://tomato_picker_description/meshes/solidworks/Link7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
- link Link7-1: mass 0.095 -> 0.0946406383916538; geometry collision mesh filename=package://tomato_picker_description/meshes/solidworks/Link7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; visual mesh filename=package://tomato_picker_description/meshes/solidworks/Link7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
- link Link7-2: mass 0.095 -> 0.0949054800343942; geometry collision mesh filename=package://tomato_picker_description/meshes/solidworks/Link7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; visual mesh filename=package://tomato_picker_description/meshes/solidworks/Link7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
- link base_link: mass 0.37451 -> 0.415436775501409
Joints:
- joint joint5: origin xyz=0.062 0.036 -0.033 rpy=1.5708 -1.5708 0 -> xyz=0.0619999999999999 0.036 -0.0330000000000007 rpy=1.5707963267949 -1.5707963267949 0
- joint joint6: limit lower=-2.094395 upper=2.094395 effort=20 velocity=5.4 -> lower=-2.0944 upper=2.0944 effort=20 velocity=5.4; origin xyz=0 -0.036 0.036 rpy=-1.5708 0 3.1416 -> xyz=0 -0.035 0.036 rpy=-1.5708 0 3.1416
- joint joint7: axis (none) -> 0 0 -1; limit (none) -> lower=0 upper=9.7674 effort=20 velocity=5.4; origin xyz=0 0 0.0605 rpy=0 0 0 -> xyz=0 0 0.051 rpy=0 0 0; type fixed -> revolute
- joint joint7-1: axis (none) -> -1 0 0; limit (none) -> lower=0 upper=0.042 effort=20 velocity=0.02322; origin xyz=-0.07 0.015 0.056 rpy=0 0 0 -> xyz=-0.068092 0.019092 0.068 rpy=-1.5708 0 0; type fixed -> prismatic
- joint joint7-2: axis (none) -> -1 0 0; limit (none) -> lower=0 upper=0.042 effort=20 velocity=0.02322; origin xyz=0.07 -0.015 0.056 rpy=0 0 0 -> xyz=0.0686415494309188 0.0190915494308821 0.0695000000001406 rpy=1.5707963267949 0 -3.14159265358979; type fixed -> prismatic
- joint tool0_joint: origin xyz=0 0 0 rpy=0 0 0 -> xyz=0 0 0.051 rpy=0 0 0
